File: CODA65.kicad_pcb (KiCad board)
At the start: 2 copper layers, 305.8 x 96.2 mm, 268 parts, among them J1 Conn_01x04, J2 Conn_01x05, SW1 SW_Push, SW2 SW_Push, SW3 RotaryEncoder_Switch, U1 RP2040, U2 W25Q128JVS, U3 74AHCT1G125, U4 XC6206PxxxMR, Y1 Crystal_GND24

Commit message: check this later
Parts:
- J1: moved to B.Cu
- moved U2 270.1 mm to (129.4, 251.6)
- moved U3 247.7 mm to (150.5, 242.2)
- moved J1 232.8 mm to (166.3, 256.4), turned to 180 degrees
- moved Y1 229.1 mm to (173.5, 220.7)
- moved U4 228.9 mm to (183.7, 238.9)
- moved C79 52.6 mm to (387.0, 209.6)

Commit message: small fixes
flipped pcb, fixed edge cut issue
Parts:
- C1, C10, C11, C12, C13, C14, C15, C16, C17, C18, C19, C2, C20, C21, C22, C23, C24, C25, C26, C27, C28, C29, C3, C30, C31, C32, C33, C34, C35, C36, C37, C38, C39, C4, C40, C41, C42, C43, C44, C45, C46, C47, C48, C49, C5, C50, C51, C52, C53, C54, C55, C56, C57, C58, C59, C6, C60, C61, C62, C63, C64, C65, C66, C67, C68, C69, C7, C70, C71, C72, C73, C74, C75, C76, C77, C78, C79, C8, C9, D1, D10, D11, D12, D13, D14, D15, D16, D17, D18, D19, D2, D20, D21, D22, D23, D24, D25, D26, D27, D28, D29, D3, D30, D31, D32, D33, D34, D35, D4, D5, D6, D7, D8, D9, J2, LED1, LED10, LED11, LED12, LED13, LED14, LED15, LED16, LED17, LED18, LED19, LED2, LED20, LED21, LED22, LED23, LED24, LED25, LED26, LED27, LED28, LED29, LED3, LED30, LED31, LED32, LED33, LED34, LED35, LED36, LED37, LED38, LED39, LED4, LED40, LED41, LED42, LED43, LED44, LED45, LED46, LED47, LED48, LED49, LED5, LED50, LED51, LED52, LED53, LED54, LED55, LED56, LED57, LED58, LED59, LED6, LED60, LED61, LED62, LED63, LED64, LED65, LED66, LED7, LED8, LED9, MX1, MX10, MX11, MX12, MX13, MX14, MX15, MX16, MX17, MX18, MX19, MX2, MX20, MX21, MX22, MX23, MX24, MX25, MX26, MX27, MX28, MX29, MX3, MX30, MX31, MX32, MX33, MX34, MX35, MX36, MX37, MX38, MX39, MX4, MX40, MX41, MX42, MX43, MX44, MX45, MX46, MX47, MX48, MX49, MX5, MX50, MX51, MX52, MX53, MX54, MX55, MX56, MX57, MX58, MX59, MX6, MX60, MX61, MX62, MX63, MX64, MX65, MX66, MX7, MX8, MX9, R1, R2, R3, R4, R5, R6, R7, R8, SW1, SW2, U1, U2, U3, U4, Y1: moved to B.Cu
- moved C18 263.9 mm to (140.2, 223.8), turned to 180 degrees
- moved C17 263.7 mm to (140.0, 218.3), turned to 180 degrees
- moved C4 256.4 mm to (146.1, 227.8), turned to 180 degrees
- moved C1 251.1 mm to (155.6, 211.9), turned to 180 degrees
- moved C5 250.6 mm to (151.6, 227.8), turned to 180 degrees
- moved C9 246.8 mm to (159.1, 228.6), turned to 180 degrees
- moved C6 246.3 mm to (155.6, 227.8), turned to 180 degrees
- moved C2 238.3 mm to (162.7, 212.7)
- moved C3 233.2 mm to (167.5, 211.9), turned to 180 degrees
- moved R8 233.0 mm to (150.8, 215.1), turned to 180 degrees
- moved C7 231.3 mm to (170.7, 228.6), turned to 180 degrees
- moved C8 230.9 mm to (173.5, 215.9), turned to 180 degrees
- moved C79 224.6 mm to (163.2, 227.8)
- moved U2 221.6 mm to (345.3, 201.6)
- moved R4 212.7 mm to (173.3, 224.6)
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
Commit message: Fixes and routing
Routed Col and Row for switches.
Fixed annotation of LEDs and caps.
Started LED matrix Routing.
Started mcu and supporting routing.
Parts:
- removed the C16 at (160.0, 147.7)
- removed the U3 at (134.1, 220.7)
- added C79: 100nF, Capacitor_SMD:C_0402_1005Metric, B.Cu at (94.8, 137.8)
- added C80: 100nF, Capacitor_SMD:C_0402_1005Metric, B.Cu at (190.1, 160.9)
- added C81: 100nF, Capacitor_SMD:C_0402_1005Metric, B.Cu at (189.1, 160.9)
- added C82: 100nF, Capacitor_SMD:C_0402_1005Metric, B.Cu at (185.8, 160.9)
- added C83: 100nF, Capacitor_SMD:C_0402_1005Metric, B.Cu at (188.1, 172.3)
- added U4: 74AHCT1G125, Package_TO_SOT_SMD:SOT-23-5, B.Cu at (91.6, 138.9)
- moved U2 148.9 mm to (196.4, 201.6), turned to 180 degrees
- moved C14 130.7 mm to (119.1, 104.8), turned to 90 degrees
- moved C18 119.4 mm to (195.3, 104.8), turned to 90 degrees
- moved R2 112.4 mm to (188.6, 158.4)
- moved R3 110.3 mm to (187.5, 158.4)
- moved R8 99.5 mm to (92.4, 134.5), turned to 90 degrees
- moved J1 80.8 mm to (227.3, 223.0)
- moved C4 74.9 mm to (183.5, 162.9)
- moved C5 74.5 mm to (195.5, 167.7), turned to 0 degrees
- moved C7 69.5 mm to (195.6, 163.7), turned to 0 degrees
- moved C6 66.1 mm to (183.0, 167.7)
- moved D7 64.0 mm to (335.0, 96.8)
- moved D34 63.6 mm to (327.3, 173.0)
- moved D1 63.3 mm to (105.1, 96.8)
- moved D13 63.3 mm to (267.0, 115.9)
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- renumbered SW1 to BOOT1, C17 to C11, C18 to C12, C11 to C13, C79 to C14, C13 to C15, C14 to C16, C15 to C17, C12 to C18, SW2 to RST1, U4 to U3
Connections:
- C12 pad 1: +3.3V -> +3V3
- D30 pad 1: Net-(D30-Pad1) -> unconnected-(D30-Pad1)
- D30 pad 2: unconnected-(D30-Pad2) -> Net-(D30-Pad2)
- D8 pad 1: unconnected-(D8-Pad1) -> Net-(D8-Pad1)
- D8 pad 2: Net-(D8-Pad2) -> unconnected-(D8-Pad2)
- LED16 pad 2: Net-(LED16-DOUT) -> Net-(LED15-DIN)
- LED17 pad 2: Net-(LED17-DOUT) -> Net-(LED16-DIN)
- LED29 pad 3: Net-(LED29-DIN) -> Net-(LED14-DOUT)
- LED30 pad 2: Net-(LED29-DIN) -> Net-(LED30-DOUT)
- LED30 pad 3: Net-(LED30-DIN) -> Net-(LED15-DOUT)
- LED31 pad 2: Net-(LED30-DIN) -> Net-(LED31-DOUT)
- LED31 pad 3: Net-(LED14-DOUT) -> Net-(LED30-DOUT)
- LED32 pad 3: Net-(LED17-DOUT) -> Net-(LED31-DOUT)
- LED44 pad 2: Net-(LED15-DIN) -> Net-(LED44-DOUT)
- LED44 pad 3: Net-(LED43-DOUT) -> Net-(LED44-DIN)
- LED45 pad 2: Net-(LED16-DIN) -> Net-(LED44-DIN)
- LED56 pad 3: Net-(LED15-DOUT) -> Net-(LED43-DOUT)
- LED57 pad 3: Net-(LED16-DOUT) -> Net-(LED44-DOUT)
- MX1 pad 2: Net-(D1-Pad2) -> Net-(D1-Pad1)
- MX10 pad 2: Net-(D5-Pad1) -> Net-(D5-Pad2)
- MX11 pad 2: Net-(D6-Pad2) -> Net-(D6-Pad1)
- MX12 pad 2: Net-(D6-Pad1) -> Net-(D6-Pad2)
- MX13 pad 2: Net-(D7-Pad2) -> Net-(D7-Pad1)
- MX14 pad 2: Net-(D7-Pad1) -> Net-(D7-Pad2)
- MX15 pad 2: Net-(D9-Pad2) -> Net-(D9-Pad1)
- MX16 pad 2: Net-(D9-Pad1) -> Net-(D9-Pad2)
- MX17 pad 2: Net-(D10-Pad2) -> Net-(D10-Pad1)
- MX18 pad 2: Net-(D10-Pad1) -> Net-(D10-Pad2)
- MX19 pad 2: Net-(D11-Pad2) -> Net-(D11-Pad1)
- MX2 pad 2: Net-(D1-Pad1) -> Net-(D1-Pad2)
- MX20 pad 2: Net-(D11-Pad1) -> Net-(D11-Pad2)
- MX21 pad 2: Net-(D12-Pad2) -> Net-(D12-Pad1)
- MX22 pad 2: Net-(D12-Pad1) -> Net-(D12-Pad2)
- MX23 pad 2: Net-(D13-Pad2) -> Net-(D13-Pad1)
- MX24 pad 2: Net-(D13-Pad1) -> Net-(D13-Pad2)
- MX25 pad 2: Net-(D14-Pad2) -> Net-(D14-Pad1)
- MX26 pad 2: Net-(D14-Pad1) -> Net-(D14-Pad2)
- MX27 pad 2: Net-(D15-Pad2) -> Net-(D15-Pad1)
- MX28 pad 2: Net-(D15-Pad1) -> Net-(D15-Pad2)
- MX3 pad 2: Net-(D2-Pad2) -> Net-(D2-Pad1)
- MX30 pad 2: Net-(D17-Pad2) -> Net-(D17-Pad1)
- MX31 pad 2: Net-(D17-Pad1) -> Net-(D17-Pad2)
- MX32 pad 2: Net-(D18-Pad2) -> Net-(D18-Pad1)
- MX33 pad 2: Net-(D18-Pad1) -> Net-(D18-Pad2)
- MX34 pad 2: Net-(D19-Pad2) -> Net-(D19-Pad1)
- MX35 pad 2: Net-(D19-Pad1) -> Net-(D19-Pad2)
- MX36 pad 2: Net-(D20-Pad2) -> Net-(D20-Pad1)
- MX37 pad 2: Net-(D20-Pad1) -> Net-(D20-Pad2)
- MX38 pad 2: Net-(D21-Pad2) -> Net-(D21-Pad1)
- MX39 pad 2: Net-(D21-Pad1) -> Net-(D21-Pad2)
- MX4 pad 2: Net-(D2-Pad1) -> Net-(D2-Pad2)
- MX40 pad 2: Net-(D22-Pad2) -> Net-(D22-Pad1)
- MX41 pad 2: Net-(D22-Pad1) -> Net-(D22-Pad2)
- MX42 pad 2: Net-(D23-Pad2) -> Net-(D23-Pad1)
- MX43 pad 2: Net-(D23-Pad1) -> Net-(D23-Pad2)
- MX44 pad 2: Net-(D24-Pad2) -> Net-(D24-Pad1)
- MX45 pad 2: Net-(D24-Pad1) -> Net-(D24-Pad2)
- MX46 pad 2: Net-(D25-Pad2) -> Net-(D25-Pad1)
- MX47 pad 2: Net-(D25-Pad1) -> Net-(D25-Pad2)
- MX48 pad 2: Net-(D26-Pad2) -> Net-(D26-Pad1)
- MX49 pad 2: Net-(D26-Pad1) -> Net-(D26-Pad2)
- MX5 pad 2: Net-(D3-Pad2) -> Net-(D3-Pad1)
- MX50 pad 2: Net-(D27-Pad2) -> Net-(D27-Pad1)
- MX51 pad 2: Net-(D27-Pad1) -> Net-(D27-Pad2)
- MX52 pad 2: Net-(D28-Pad2) -> Net-(D28-Pad1)
- MX53 pad 2: Net-(D28-Pad1) -> Net-(D28-Pad2)
- MX54 pad 2: Net-(D29-Pad2) -> Net-(D29-Pad1)
- MX55 pad 2: Net-(D29-Pad1) -> Net-(D29-Pad2)
- MX56 pad 2: Net-(D30-Pad1) -> Net-(D30-Pad2)
- MX57 pad 2: Net-(D31-Pad2) -> Net-(D31-Pad1)
- MX58 pad 2: Net-(D31-Pad1) -> Net-(D31-Pad2)
- MX59 pad 2: Net-(D32-Pad2) -> Net-(D32-Pad1)
- MX6 pad 2: Net-(D3-Pad1) -> Net-(D3-Pad2)
- MX60 pad 2: Net-(D32-Pad1) -> Net-(D32-Pad2)
- MX61 pad 2: Net-(D33-Pad2) -> Net-(D33-Pad1)
- MX62 pad 2: Net-(D33-Pad1) -> Net-(D33-Pad2)
- MX63 pad 2: Net-(D34-Pad2) -> Net-(D34-Pad1)
- MX64 pad 2: Net-(D34-Pad1) -> Net-(D34-Pad2)
- MX65 pad 2: Net-(D35-Pad2) -> Net-(D35-Pad1)
- MX66 pad 2: Net-(D35-Pad1) -> Net-(D35-Pad2)
- MX7 pad 2: Net-(D4-Pad2) -> Net-(D4-Pad1)
- MX8 pad 2: Net-(D4-Pad1) -> Net-(D4-Pad2)
- MX9 pad 2: Net-(D5-Pad2) -> Net-(D5-Pad1)
- SW3 pad S1: Net-(D8-Pad2) -> Net-(D8-Pad1)
- U3 pad 2: +3.3V -> +3V3
Routing:
- net ROW0: track 0.00 -> 297.2 mm
- net ROW1: track 0.00 -> 260.1 mm
- net ROW2: track 0.00 -> 250.8 mm
- net ROW3: track 0.00 -> 231.0 mm
- net ROW4: track 0.00 -> 130.2 mm
- net COL1: track 0.00 -> 114.9 mm
- net COL3: track 0.00 -> 113.6 mm
- net COL2: track 0.00 -> 113.5 mm
- net COL11: track 0.00 -> 108.7 mm
- net COL10: track 0.00 -> 101.6 mm
- net COL6: track 0.00 -> 101.5 mm
- net COL9: track 0.00 -> 99.4 mm
- net Col0: track 0.00 -> 93.5 mm
- net COL13: track 0.00 -> 81.6 mm
- net COL14: track 0.00 -> 80.6 mm
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Other:
- board size 305.8 x 96.2 mm -> 303.2 x 93.7 mm

Commit message: LED Routing
LED Data matrix moslty routed out besides home runs.
Parts:
- moved C29 10.5 mm to (139.7, 119.1), turned to -90 degrees
- moved C67 10.4 mm to (332.6, 157.2), turned to -90 degrees
- moved C65 10.4 mm to (287.3, 157.2), turned to -90 degrees
- moved C60 10.4 mm to (192.1, 157.3), turned to -90 degrees
- moved C66 10.3 mm to (306.4, 157.2), turned to -90 degrees
- moved C61 10.3 mm to (211.1, 157.3), turned to -90 degrees
- moved C28 10.3 mm to (120.7, 119.1), turned to -90 degrees
- moved C33 10.3 mm to (215.9, 119.1), turned to -90 degrees
- moved C57 10.3 mm to (134.9, 157.3), turned to -90 degrees
- moved C62 10.3 mm to (230.2, 157.3), turned to -90 degrees
- moved C39 10.3 mm to (330.2, 118.9), turned to -90 degrees
- moved C34 10.3 mm to (234.9, 119.1), turned to -90 degrees
- moved C56 10.2 mm to (104.0, 157.3), turned to -90 degrees
- moved C35 10.2 mm to (254.0, 118.7), turned to -90 degrees
- moved C58 10.2 mm to (154.0, 157.3), turned to -90 degrees
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Routing:
- net Net-(LED42-DOUT): track 0.00 -> 26.1 mm
- net Net-(LED44-DIN): track 0.00 -> 26.1 mm
- net Net-(LED41-DOUT): track 0.00 -> 26.1 mm
- net Net-(LED55-DIN): track 0.00 -> 21.4 mm
- net Net-(LED30-DOUT): track 0.00 -> 21.4 mm
- net Net-(LED63-DOUT): track 0.00 -> 21.4 mm
- net Net-(LED54-DIN): track 0.00 -> 21.4 mm
- net Net-(LED28-DIN): track 0.00 -> 19.0 mm
- net Net-(LED27-DIN): track 0.00 -> 19.0 mm
- net Net-(LED15-DIN): track 0.00 -> 19.0 mm
- net Net-(LED58-DOUT): track 0.00 -> 16.6 mm
- net Net-(LED62-DOUT): track 0.00 -> 16.6 mm
- net Net-(LED57-DOUT): track 0.00 -> 16.6 mm
- net Net-(LED65-DOUT): track 0.00 -> 14.2 mm
- net Net-(LED64-DOUT): track 0.00 -> 14.2 mm
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